Commit message: component updated

File: system_description/urdf/camera_holder.urdf.xacro (robot description, xacro)
@@ -12,5 +12,5 @@
         <origin rpy="0 0 0" xyz="0 0 0"/>
         <geometry>
-          <mesh filename="package://erik_description/meshes/skamera_ur_new.stl" scale="0.001 0.001 0.001"/>
+          <mesh filename="package://system_description/meshes/skamera_ur_new.stl" scale="0.001 0.001 0.001"/>
         </geometry>
         <!-- <material name="LightGrey">
@@ -24,5 +24,5 @@
         <origin rpy="0 0 0" xyz="0 0 0"/>
         <geometry>
-          <mesh filename="package://erik_description/meshes/skamera_ur_new.stl" scale="0.001 0.001 0.001"/>
+          <mesh filename="package://system_description/meshes/skamera_ur_new.stl" scale="0.001 0.001 0.001"/>
         </geometry>
       </collision>

File: system_description/urdf/gripper_bracket.urdf.xacro (robot description, xacro)
@@ -16,5 +16,5 @@
         <origin rpy="0 0 0" xyz="0 0 0"/>
         <geometry>
-          <mesh filename="package://erik_description/meshes/gripper_bracket_with_screws.stl" scale="0.001 0.001 0.001"/>
+          <mesh filename="package://system_description/meshes/gripper_bracket_with_screws.stl" scale="0.001 0.001 0.001"/>
         </geometry>
         <material name="LightGrey">
@@ -25,5 +25,5 @@
         <origin rpy="0 0 0" xyz="0 0 0"/>
         <geometry>
-          <mesh filename="package://erik_description/meshes/gripper_bracket_with_screws.stl" scale="0.001 0.001 0.001"/>
+          <mesh filename="package://system_description/meshes/gripper_bracket_with_screws.stl" scale="0.001 0.001 0.001"/>
         </geometry>
       </collision>

File: system_description/urdf/manipulator.urdf.xacro (robot description, xacro)
@@ -8,7 +8,7 @@
   <xacro:include filename="$(find ur_description)/urdf/ur.urdf.xacro" ur_type="ur3e" />
   <!-- camera holder for d455 -->
-  <xacro:include filename="$(find erik_description)/urdf/simple_camera_holder_new.urdf.xacro" />
+  <xacro:include filename="$(find system_description)/urdf/simple_camera_holder_new.urdf.xacro" />
   <!-- gripper bracket -->
-  <xacro:include filename="$(find erik_description)/urdf/gripper_bracket.urdf.xacro" />
+  <xacro:include filename="$(find system_description)/urdf/gripper_bracket.urdf.xacro" />
   <!-- intel realsense camera  -->
   <xacro:include filename="$(find realsense2_description)/urdf/_d455.urdf.xacro" />
