Commit message: namespace fixing

File: system_description/urdf/closed_control_loop.urdf.xacro (robot description, xacro)
@@ -2,15 +2,15 @@
 <robot xmlns:xacro="http://ros.org/wiki/xacro"
        xmlns:rcl="urn:robot-control-loop"
-       xmlns:nw="urn:network"
-       xmlns:nt="urn:network-topology"
+       xmlns:nw="urn:robot-network"
+       xmlns:nt="urn:robot-network-topology"
        xmlns:l1t="urn:layer1"
        xmlns:l2t="urn:layer2"
        name="closed-control-loop">
-    <xacro:macro name="closed-control-loop" params="control_loop_id containing_link_ids latency cycle_time frequency payload_capacity reach end_effector_type safety_features maintenance_requirements environment safety_standard_compliance">
+    <xacro:macro name="closed-control-loop" params="control_loop_id supporting_links latency cycle_time frequency payload_capacity reach safety_features maintenance_requirements environment safety_standard_compliance">
         <yang>
             <!-- robot-control-loop -->
             <rcl:control-loops>
                 <rcl:control-loop-id>${control_loop_id}</rcl:control-loop-id>
-                <containing-link-ids>${containing_link_ids}</containing-link-ids>
+                <containing-link-ids>${supporting_links}</containing-link-ids>
                 <latency>${latency}</latency>
                 <cycle-time>${cycle_time}</cycle-time>
@@ -18,5 +18,5 @@
                 <payload-capacity>${payload_capacity}</payload-capacity>
                 <reach>${reach}</reach>
-                <end-effector-type>${end_effector_type}</end-effector-type>
+                <!-- <end-effector-type>${end_effector_type}</end-effector-type> -->
                 <safety-features>${safety_features}</safety-features>
                 <maintenance-requirements>${maintenance_requirements}</maintenance-requirements>

File: system_description/urdf/connections.urdf.xacro (robot description, xacro)
@@ -1,10 +1,10 @@
 <?xml version="1.0"?>
 <robot xmlns:xacro="http://ros.org/wiki/xacro"
-       xmlns:nw="urn:network"
-       xmlns:nt="urn:network-topology"
+       xmlns:nw="urn:robot-network"
+       xmlns:nt="urn:robot-network-topology"
        xmlns:l1t="urn:layer1"
        xmlns:l2t="urn:layer2"
        name="topology-link">
-    <xacro:macro name="topology-link" params="src_node src_tp dst_node dst_tp conn_type">
+    <xacro:macro name="topology-link" params="src_node src_tp dst_node dst_tp conn_type reconfig">
         <yang>
             <!-- robot-network-topology-link -->
@@ -14,4 +14,5 @@
                     <l1t:l1-link-attributes>
                         <type>${conn_type}</type>
+                        <reconfig>${reconfig}</reconfig>
                     </l1t:l1-link-attributes>
                     <nt:source>

File: system_description/urdf/manipulator.urdf.xacro (robot description, xacro)
@@ -47,5 +47,5 @@
   </xacro:sensor_d455>
 <!-- Connection/link descriptions -->
-  <yang xmlns:nw="urn:network">
+  <yang xmlns:nw="urn:robot-network">
     <!-- link between d455cam and nuc -->
     <connection name="nuc-sensor_d455" type="wired" dev1="nuc" dev2="sensor_d455" />
