Commit message: namespaces restructured

File: system_description/urdf/connections.urdf.xacro (robot description, xacro)
@@ -1,29 +1,29 @@
 <?xml version="1.0"?>
 <robot xmlns:xacro="http://ros.org/wiki/xacro"
-       xmlns:nw="urn:robot-network"
-       xmlns:nt="urn:robot-network-topology"
-       xmlns:l1t="urn:layer1"
-       xmlns:l2t="urn:layer2"
+       xmlns:robot-network-topology="urn:ietf:params:xml:ns:yang:robot-network-topology"
+       xmlns:layer1="urn:ietf:params:xml:ns:yang:layer1"
        name="topology-link">
-    <xacro:macro name="topology-link" params="src_node src_tp dst_node dst_tp conn_type reconfig">
+    <xacro:macro name="topology-link" params="topology_link_id src_node src_tp dst_node dst_tp conn_type reconfig">
         <yang>
             <!-- robot-network-topology-link -->
-            <nw:network>
-                <nw:robot-network-topology-link>
-                    <nt:link-id>${src_node}-${dst_node}-link</nt:link-id>
-                    <l1t:l1-link-attributes>
+            <network>
+            <network-id>topology_level</network-id>
+                <robot-network-topology:link>
+                    <link-id>${topology_link_id}</link-id>
+                    <robot-network-topology:link-id>${src_node}-${dst_node}-link</robot-network-topology:link-id>
+                    <layer1:l1-link-attributes>
                         <type>${conn_type}</type>
                         <reconfig>${reconfig}</reconfig>
-                    </l1t:l1-link-attributes>
-                    <nt:source>
+                    </layer1:l1-link-attributes>
+                    <source>
                         <source-node>${src_node}</source-node>
                         <source-tp>${src_tp}</source-tp>
-                    </nt:source>
-                    <nt:destination>
+                    </source>
+                    <destination>
                         <dest-node>${dst_node}</dest-node>
                         <dest-tp>${dst_tp}</dest-tp>
-                    </nt:destination>
-                </nw:robot-network-topology-link>
-            </nw:network>
+                    </destination>
+                </robot-network-topology:link>
+            </network>
         </yang>
     </xacro:macro>

Commit message: topology-link-id not required

File: system_description/urdf/connections.urdf.xacro (robot description, xacro)
@@ -4,5 +4,5 @@
        xmlns:layer1="urn:ietf:params:xml:ns:yang:layer1"
        name="topology-link">
-    <xacro:macro name="topology-link" params="topology_link_id src_node src_tp dst_node dst_tp conn_type reconfig">
+    <xacro:macro name="topology-link" params="src_node src_tp dst_node dst_tp conn_type reconfig">
         <yang>
             <!-- robot-network-topology-link -->
@@ -10,5 +10,4 @@
             <network-id>topology_level</network-id>
                 <robot-network-topology:link>
-                    <link-id>${topology_link_id}</link-id>
                     <robot-network-topology:link-id>${src_node}-${dst_node}-link</robot-network-topology:link-id>
                     <layer1:l1-link-attributes>

File: system_description/urdf/robot_system_description.urdf.xacro (robot description, xacro)
@@ -141,15 +141,15 @@
    <!-- link radiodot with world -->
    <xacro:radiodot parent="world"/>
-   <xacro:topology-link topology_link_id="1" src_node="poe-switch" src_tp="eth_1" dst_node="mikrotik" dst_tp="eth_1" conn_type="wired" reconfig="hw_supported"/>
-   <xacro:topology-link topology_link_id="2" src_node="mikrotik" src_tp="eth_2" dst_node="rpi4" dst_tp="eth_1" conn_type="wired" reconfig="hw_supported"/>
-   <xacro:topology-link topology_link_id="3" src_node="realsense-d455i" src_tp="usb_1" dst_node="nuc" dst_tp="usb_1" conn_type="wired" reconfig="hw_supported"/>
-   <xacro:topology-link topology_link_id="4" src_node="nuc" src_tp="eth_1" dst_node="poe-switch" dst_tp="eth_2" conn_type="wired" reconfig="hw_supported"/>
-   <xacro:topology-link topology_link_id="5" src_node="rg2ft-computebox" src_tp="eth_1" dst_node="poe-switch" dst_tp="eth_3" conn_type="wired" reconfig="hw_supported"/>
-   <xacro:topology-link topology_link_id="6" src_node="rg2ft-computebox" src_tp="prop_1" dst_node="rg2ft-gripper" dst_tp="prop_1" conn_type="wired" reconfig="hw_supported"/>
-   <xacro:topology-link topology_link_id="7" src_node="ur3e-controlbox" src_tp="eth_1" dst_node="poe-switch" dst_tp="eth_4" conn_type="wired" reconfig="hw_supported"/>
-   <xacro:topology-link topology_link_id="8" src_node="ur3e-controlbox" src_tp="prop_1" dst_node="ur3e-arm" dst_tp="prop_1" conn_type="wired" reconfig="hw_supported"/>
-   <xacro:topology-link topology_link_id="9" src_node="5g-modem" src_tp="usb_1" dst_node="rpi4" dst_tp="usb_1" conn_type="wired" reconfig="hw_supported"/>
-   <xacro:topology-link topology_link_id="10" src_node="5g-modem" src_tp="wireless_1" dst_node="5g-dot" dst_tp="wireless_1" conn_type="wireless" reconfig="sw_supported"/>
-   <xacro:topology-link topology_link_id="11" src_node="5g-dot" src_tp="eth_1" dst_node="flightrack" dst_tp="eth_1" conn_type="wired" reconfig="sw_supported"/>
+   <xacro:topology-link src_node="poe-switch" src_tp="eth_1" dst_node="mikrotik" dst_tp="eth_1" conn_type="wired" reconfig="hw_supported"/>
+   <xacro:topology-link src_node="mikrotik" src_tp="eth_2" dst_node="rpi4" dst_tp="eth_1" conn_type="wired" reconfig="hw_supported"/>
+   <xacro:topology-link src_node="realsense-d455i" src_tp="usb_1" dst_node="nuc" dst_tp="usb_1" conn_type="wired" reconfig="hw_supported"/>
+   <xacro:topology-link src_node="nuc" src_tp="eth_1" dst_node="poe-switch" dst_tp="eth_2" conn_type="wired" reconfig="hw_supported"/>
+   <xacro:topology-link src_node="rg2ft-computebox" src_tp="eth_1" dst_node="poe-switch" dst_tp="eth_3" conn_type="wired" reconfig="hw_supported"/>
+   <xacro:topology-link src_node="rg2ft-computebox" src_tp="prop_1" dst_node="rg2ft-gripper" dst_tp="prop_1" conn_type="wired" reconfig="hw_supported"/>
+   <xacro:topology-link src_node="ur3e-controlbox" src_tp="eth_1" dst_node="poe-switch" dst_tp="eth_4" conn_type="wired" reconfig="hw_supported"/>
+   <xacro:topology-link src_node="ur3e-controlbox" src_tp="prop_1" dst_node="ur3e-arm" dst_tp="prop_1" conn_type="wired" reconfig="hw_supported"/>
+   <xacro:topology-link src_node="5g-modem" src_tp="usb_1" dst_node="rpi4" dst_tp="usb_1" conn_type="wired" reconfig="hw_supported"/>
+   <xacro:topology-link src_node="5g-modem" src_tp="wireless_1" dst_node="5g-dot" dst_tp="wireless_1" conn_type="wireless" reconfig="sw_supported"/>
+   <xacro:topology-link src_node="5g-dot" src_tp="eth_1" dst_node="flightrack" dst_tp="eth_1" conn_type="wired" reconfig="sw_supported"/>
    <xacro:closed-control-loop
       control_loop_id="1"
