Commit message: namespaces updated, interfaces added

File: network-components/nuc_description/urdf/nuc.urdf.xacro (robot description, xacro)
@@ -1,6 +1,6 @@
 <?xml version="1.0"?>
 <robot xmlns:xacro="http://ros.org/wiki/xacro"
-       xmlns:nw="urn:network"
-       xmlns:nt="urn:network-topology"
+       xmlns:nw="urn:robot-network"
+       xmlns:nt="urn:robot-network-topology"
        xmlns:l1t="urn:layer1"
        xmlns:l2t="urn:layer2"
@@ -9,5 +9,5 @@
     <xacro:include filename="$(find interface-description)/urdf/usb30.urdf.xacro"/>
     <xacro:include filename="$(find interface-description)/urdf/wifi5.urdf.xacro"/>
-    <xacro:macro name="nuc" params="parent L2_network_id:=Data_Link L1_network_id:=Physical L2_id:=NUC_L2 L1_id:=NUC_L1">
+    <xacro:macro name="nuc" params="parent L2_network_id:=network_level L1_network_id:=device_level L2_id:=nuc_L2 L1_id:=nuc_L1">
     <!-- <xacro:macro name="nuc" params="parent L1_id L2_id L1_network_id L2_network_id"> -->
         <joint name="nuc_joint" type="fixed">
@@ -50,4 +50,8 @@
                     </nw:supporting-node>
                     <xacro:usb30_L2 id="usb_1" supporting_network="${L1_network_id}" supporting_node="${L1_id}" supporting_tp="usb_1"/>
+                    <xacro:usb30_L2 id="usb_2" supporting_network="${L1_network_id}" supporting_node="${L1_id}" supporting_tp="usb_2"/>
+                    <xacro:usb30_L2 id="usb_3" supporting_network="${L1_network_id}" supporting_node="${L1_id}" supporting_tp="usb_3"/>
+                    <xacro:usb30_L2 id="usb_4" supporting_network="${L1_network_id}" supporting_node="${L1_id}" supporting_tp="usb_3"/>
+                    <xacro:usb30_L2 id="usb_5" supporting_network="${L1_network_id}" supporting_node="${L1_id}" supporting_tp="usb_3"/>
                     <xacro:cat6_L2 id="eth_1" supporting_network="${L1_network_id}" supporting_node="${L1_id}" supporting_tp="eth_1"/>
                     <xacro:wifi5_L2 id="wireless_1" supporting_network="${L1_network_id}" supporting_node="${L1_id}" supporting_tp="wireless_1"/>
@@ -65,7 +69,11 @@
                         <l1t:device-type>pc</l1t:device-type>
                     </l1t:l1-node-attributes>
-                    <xacro:usb30_L1 id="usb_1"/>
-                    <xacro:cat6_L1 id="eth_1"/>
-                    <xacro:wifi5_L1 id="wireless_1"/>
+                    <xacro:usb30_L1 id="usb_1" connector_type="usb-std_A" connector_format="female"/>
+                    <xacro:usb30_L1 id="usb_2" connector_type="usb-std_A" connector_format="female"/>
+                    <xacro:usb30_L1 id="usb_3" connector_type="usb-std_A" connector_format="female"/>
+                    <xacro:usb30_L1 id="usb_4" connector_type="usb-type_C" connector_format="female"/>
+                    <xacro:usb30_L1 id="usb_5" connector_type="usb-type_C" connector_format="female"/>
+                    <xacro:cat6_L1 id="eth_1" connector_type="rj45" connector_format="female"/>
+                    <!-- <xacro:wifi5_L1 id="wireless_1" connector-type="wireless" connector_format="wireless"/> -->
                 </nw:node>
             </nw:network>
