Commit message: yang layer update

File: network-components/interface-description/urdf/cat5e.urdf.xacro (robot description, xacro)
@@ -1,6 +1,6 @@
 <?xml version="1.0" encoding="UTF-8" ?>
 <robot xmlns:xacro="http://ros.org/wiki/xacro"
-       xmlns:nw="urn:network"
-       xmlns:nt="urn:network-topology"
+       xmlns:nw="urn:robot-network"
+       xmlns:nt="urn:robot-network-topology"
        xmlns:l1t="urn:layer1"
        xmlns:l2t="urn:layer2"
@@ -21,12 +21,4 @@
     <xacro:property name="cat5e_scalability" value="${cat5e_props['wired-connection']['scalability']}"/>
     <xacro:property name="cat5e_security_level" value="${cat5e_props['wired-connection']['security-level']}"/>
-    <xacro:macro name="cat5e_L1" params="id">
-        <nt:termination-point>
-            <nt:tp-id>${id}</nt:tp-id>
-            <l1t:l1-termination-point-attributes>
-                <l1t:intertface-type>cat5e</l1t:intertface-type>
-            </l1t:l1-termination-point-attributes>
-        </nt:termination-point>
-    </xacro:macro>
     <xacro:macro name="cat5e_L2" params="id supporting_network supporting_node supporting_tp">
         <nt:termination-point>
@@ -43,3 +35,12 @@
         </nt:termination-point>
     </xacro:macro>
+    <xacro:macro name="cat5e_L1" params="id connector_type connector_format">
+        <nt:termination-point>
+            <nt:tp-id>${id}</nt:tp-id>
+            <l1t:l1-termination-point-attributes>
+                <l1t:connector-type>${connector_type}</l1t:connector-type>
+                <l1t:connector-format>${connector_format}</l1t:connector-format>
+            </l1t:l1-termination-point-attributes>
+        </nt:termination-point>
+    </xacro:macro>
 </robot>

File: network-components/interface-description/urdf/cat6.urdf.xacro (robot description, xacro)
@@ -1,6 +1,6 @@
 <?xml version="1.0" encoding="UTF-8" ?>
 <robot xmlns:xacro="http://ros.org/wiki/xacro"
-       xmlns:nw="urn:network"
-       xmlns:nt="urn:network-topology"
+       xmlns:nw="urn:robot-network"
+       xmlns:nt="urn:robot-network-topology"
        xmlns:l1t="urn:layer1"
        xmlns:l2t="urn:layer2"
@@ -21,11 +21,27 @@
     <xacro:property name="cat6_scalability" value="${cat6_props['wired-connection']['scalability']}"/>
     <xacro:property name="cat6_security_level" value="${cat6_props['wired-connection']['security-level']}"/>
-    <xacro:macro name="cat6_L1" params="id">
-        <nt:termination-point>
-            <nt:tp-id>${id}</nt:tp-id>
-            <l1t:l1-termination-point-attributes>
-                <l1t:intertface-type>cat6</l1t:intertface-type>
-            </l1t:l1-termination-point-attributes>
-        </nt:termination-point>
+    <xacro:macro name="cat6" params="parent L2_network_id L1_network_id L2_id:=cat6_L2 L1_id:=cat6_L1">
+        <joint name="cat6_joint" type="fixed">
+            <origin xyz="-1 1 0" rpy="0 0 0" />
+            <parent link="${parent}"/>
+            <child link="cat6_link"/>
+        </joint>
+        <link name="cat6_link">
+            <visual>
+                <origin rpy="0 0 0" xyz="0 0 0"/>
+                <geometry>
+                <mesh filename="package://interface_description/meshes/rj45_female.stl" scale="0.001 0.001 0.001"/>
+                </geometry>
+                <material name="LightGrey">
+                <color rgba="0.7 0.7 0.7 1.0"/>
+                </material>
+            </visual>
+            <collision>
+                <origin xyz="0 0 0" rpy="0 0 0"/>
+                <geometry>
+                <mesh filename="package://interface_description/meshes/rj45_female.stl" scale="0.001 0.001 0.001"/>
+                </geometry>
+            </collision>
+        </link>
     </xacro:macro>
     <xacro:macro name="cat6_L2" params="id supporting_network supporting_node supporting_tp">
@@ -43,3 +59,12 @@
         </nt:termination-point>
     </xacro:macro>
+    <xacro:macro name="cat6_L1" params="id connector_type connector_format">
+        <nt:termination-point>
+            <nt:tp-id>${id}</nt:tp-id>
+            <l1t:l1-termination-point-attributes>
+                <l1t:connector-type>${connector_type}</l1t:connector-type>
+                <l1t:connector-format>${connector_format}</l1t:connector-format>
+            </l1t:l1-termination-point-attributes>
+        </nt:termination-point>
+    </xacro:macro>
 </robot>

File: network-components/interface-description/urdf/nw_5g_rel15.urdf.xacro (robot description, xacro)
@@ -1,6 +1,6 @@
 <?xml version="1.0" encoding="UTF-8" ?>
 <robot xmlns:xacro="http://ros.org/wiki/xacro"
-       xmlns:nw="urn:network"
-       xmlns:nt="urn:network-topology"
+       xmlns:nw="urn:robot-network"
+       xmlns:nt="urn:robot-network-topology"
        xmlns:l1t="urn:layer1"
        xmlns:l2t="urn:layer2"
@@ -21,13 +21,5 @@
     <xacro:property name="nw_5g_rel15_scalability" value="${nw_5g_rel15_props['wireless-connection']['scalability']}"/>
     <xacro:property name="nw_5g_rel15_security_level" value="${nw_5g_rel15_props['wireless-connection']['security-level']}"/>
-    <xacro:macro name="nw-5g-rel15_L1" params="id">
-        <nt:termination-point>
-            <nt:tp-id>${id}</nt:tp-id>
-            <l1t:l1-termination-point-attributes>
-                <l1t:intertface-type>nw_5g_rel15</l1t:intertface-type>
-            </l1t:l1-termination-point-attributes>
-        </nt:termination-point>
-    </xacro:macro>
-    <xacro:macro name="nw-5g-rel15_L2" params="id supporting_network supporting_node supporting_tp">
+    <xacro:macro name="nw_5g_rel15_L2" params="id supporting_network supporting_node supporting_tp">
         <nt:termination-point>
             <nt:tp-id>${id}</nt:tp-id>
@@ -43,3 +35,12 @@
         </nt:termination-point>
     </xacro:macro>
+    <xacro:macro name="nw_5g_rel15_L1" params="id connector_type connector_format">
+        <nt:termination-point>
+            <nt:tp-id>${id}</nt:tp-id>
+            <l1t:l1-termination-point-attributes>
+                <l1t:connector-type>${connector_type}</l1t:connector-type>
+                <l1t:connector-format>${connector_format}</l1t:connector-format>
+            </l1t:l1-termination-point-attributes>
+        </nt:termination-point>
+    </xacro:macro>
 </robot>

File: network-components/interface-description/urdf/usb20.urdf.xacro (robot description, xacro)
@@ -1,6 +1,6 @@
 <?xml version="1.0" encoding="UTF-8" ?>
 <robot xmlns:xacro="http://ros.org/wiki/xacro"
-       xmlns:nw="urn:network"
-       xmlns:nt="urn:network-topology"
+       xmlns:nw="urn:robot-network"
+       xmlns:nt="urn:robot-network-topology"
        xmlns:l1t="urn:layer1"
        xmlns:l2t="urn:layer2"
@@ -21,12 +21,4 @@
     <xacro:property name="usb20_scalability" value="${usb20_props['wired-connection']['scalability']}"/>
     <xacro:property name="usb20_security_level" value="${usb20_props['wired-connection']['security-level']}"/>
-    <xacro:macro name="usb20_L1" params="id">
-        <nt:termination-point>
-            <nt:tp-id>${id}</nt:tp-id>
-            <l1t:l1-termination-point-attributes>
-                <l1t:interface-type>usb20</l1t:interface-type>
-            </l1t:l1-termination-point-attributes>
-        </nt:termination-point>
-    </xacro:macro>
     <xacro:macro name="usb20_L2" params="id supporting_network supporting_node supporting_tp">
         <nt:termination-point>
@@ -43,3 +35,12 @@
         </nt:termination-point>
     </xacro:macro>
+    <xacro:macro name="usb20_L1" params="id connector_type connector_format">
+        <nt:termination-point>
+            <nt:tp-id>${id}</nt:tp-id>
+            <l1t:l1-termination-point-attributes>
+                <l1t:connector-type>${connector_type}</l1t:connector-type>
+                <l1t:connector-format>${connector_format}</l1t:connector-format>
+            </l1t:l1-termination-point-attributes>
+        </nt:termination-point>
+    </xacro:macro>
 </robot>

File: network-components/interface-description/urdf/usb30.urdf.xacro (robot description, xacro)
@@ -1,6 +1,6 @@
 <?xml version="1.0" encoding="UTF-8" ?>
 <robot xmlns:xacro="http://ros.org/wiki/xacro"
-       xmlns:nw="urn:network"
-       xmlns:nt="urn:network-topology"
+       xmlns:nw="urn:robot-network"
+       xmlns:nt="urn:robot-network-topology"
        xmlns:l1t="urn:layer1"
        xmlns:l2t="urn:layer2"
@@ -21,12 +21,4 @@
     <xacro:property name="usb30_scalability" value="${usb30_props['wired-connection']['scalability']}"/>
     <xacro:property name="usb30_security_level" value="${usb30_props['wired-connection']['security-level']}"/>
-    <xacro:macro name="usb30_L1" params="id">
-        <nt:termination-point>
-            <nt:tp-id>${id}</nt:tp-id>
-            <l1t:l1-termination-point-attributes>
-                <l1t:interface-type>usb30</l1t:interface-type>
-            </l1t:l1-termination-point-attributes>
-        </nt:termination-point>
-    </xacro:macro>
     <xacro:macro name="usb30_L2" params="id supporting_network supporting_node supporting_tp">
         <nt:termination-point>
@@ -43,3 +35,12 @@
         </nt:termination-point>
     </xacro:macro>
+    <xacro:macro name="usb30_L1" params="id connector_type connector_format">
+        <nt:termination-point>
+            <nt:tp-id>${id}</nt:tp-id>
+            <l1t:l1-termination-point-attributes>
+                <l1t:connector-type>${connector_type}</l1t:connector-type>
+                <l1t:connector-format>${connector_format}</l1t:connector-format>
+            </l1t:l1-termination-point-attributes>
+        </nt:termination-point>
+    </xacro:macro>
 </robot>

File: network-components/interface-description/urdf/wifi4.urdf.xacro (robot description, xacro)
@@ -1,6 +1,6 @@
 <?xml version="1.0" encoding="UTF-8" ?>
 <robot xmlns:xacro="http://ros.org/wiki/xacro"
-       xmlns:nw="urn:network"
-       xmlns:nt="urn:network-topology"
+       xmlns:nw="urn:robot-network"
+       xmlns:nt="urn:robot-network-topology"
        xmlns:l1t="urn:layer1"
        xmlns:l2t="urn:layer2"
@@ -21,12 +21,5 @@
     <xacro:property name="wifi4_scalability" value="${wifi4_props['wireless-connection']['scalability']}"/>
     <xacro:property name="wifi4_security_level" value="${wifi4_props['wireless-connection']['security-level']}"/>
-    <xacro:macro name="wifi4_L1" params="id">
-        <nt:termination-point>
-            <nt:tp-id>${id}</nt:tp-id>
-            <l1t:l1-termination-point-attributes>
-                <l1t:intertface-type>wifi4</l1t:intertface-type>
-            </l1t:l1-termination-point-attributes>
-        </nt:termination-point>
-    </xacro:macro>
+    <xacro:macro name="wifi4" params="parent L2_network_id L1_network_id L2_id:=wifi4_L2 L1_id:=wifi4_L1"/>
     <xacro:macro name="wifi4_L2" params="id supporting_network supporting_node supporting_tp">
         <nt:termination-point>
@@ -43,3 +36,12 @@
         </nt:termination-point>
     </xacro:macro>
+    <xacro:macro name="wifi4_L1" params="id connector_type connector_format">
+        <nt:termination-point>
+            <nt:tp-id>${id}</nt:tp-id>
+            <l1t:l1-termination-point-attributes>
+                <l1t:connector-type>${connector_type}</l1t:connector-type>
+                <l1t:connector-format>${connector_format}</l1t:connector-format>
+            </l1t:l1-termination-point-attributes>
+        </nt:termination-point>
+    </xacro:macro>
 </robot>

File: network-components/interface-description/urdf/wifi5.urdf.xacro (robot description, xacro)
@@ -1,6 +1,6 @@
 <?xml version="1.0" encoding="UTF-8" ?>
 <robot xmlns:xacro="http://ros.org/wiki/xacro"
-       xmlns:nw="urn:network"
-       xmlns:nt="urn:network-topology"
+       xmlns:nw="urn:robot-network"
+       xmlns:nt="urn:robot-network-topology"
        xmlns:l1t="urn:layer1"
        xmlns:l2t="urn:layer2"
@@ -21,12 +21,5 @@
     <xacro:property name="wifi5_scalability" value="${wifi5_props['wireless-connection']['scalability']}"/>
     <xacro:property name="wifi5_security_level" value="${wifi5_props['wireless-connection']['security-level']}"/>
-    <xacro:macro name="wifi5_L1" params="id">
-        <nt:termination-point>
-            <nt:tp-id>${id}</nt:tp-id>
-            <l1t:l1-termination-point-attributes>
-                <l1t:intertface-type>wifi5</l1t:intertface-type>
-            </l1t:l1-termination-point-attributes>
-        </nt:termination-point>
-    </xacro:macro>
+    <xacro:macro name="wifi5" params="parent L2_network_id L1_network_id L2_id:=wifi5_L2 L1_id:=wifi5_L1"/>
     <xacro:macro name="wifi5_L2" params="id supporting_network supporting_node supporting_tp">
         <nt:termination-point>
@@ -43,3 +36,12 @@
         </nt:termination-point>
     </xacro:macro>
+    <xacro:macro name="wifi5_L1" params="id connector_type connector_format">
+        <nt:termination-point>
+            <nt:tp-id>${id}</nt:tp-id>
+            <l1t:l1-termination-point-attributes>
+                <l1t:connector-type>${connector_type}</l1t:connector-type>
+                <l1t:connector-format>${connector_format}</l1t:connector-format>
+            </l1t:l1-termination-point-attributes>
+        </nt:termination-point>
+    </xacro:macro>
 </robot>

File: network-components/interface-description/urdf/wifi6.urdf.xacro (robot description, xacro)
@@ -1,6 +1,6 @@
 <?xml version="1.0" encoding="UTF-8" ?>
 <robot xmlns:xacro="http://ros.org/wiki/xacro"
-       xmlns:nw="urn:network"
-       xmlns:nt="urn:network-topology"
+       xmlns:nw="urn:robot-network"
+       xmlns:nt="urn:robot-network-topology"
        xmlns:l1t="urn:layer1"
        xmlns:l2t="urn:layer2"
@@ -21,12 +21,5 @@
     <xacro:property name="wifi6_scalability" value="${wifi6_props['wireless-connection']['scalability']}"/>
     <xacro:property name="wifi6_security_level" value="${wifi6_props['wireless-connection']['security-level']}"/>
-    <xacro:macro name="wifi6_L1" params="id">
-        <nt:termination-point>
-            <nt:tp-id>${id}</nt:tp-id>
-            <l1t:l1-termination-point-attributes>
-                <l1t:intertface-type>wifi6</l1t:intertface-type>
-            </l1t:l1-termination-point-attributes>
-        </nt:termination-point>
-    </xacro:macro>
+    <xacro:macro name="wifi6" params="parent L2_network_id L1_network_id L2_id:=wifi6_L2 L1_id:=wifi6_L1"/>
     <xacro:macro name="wifi6_L2" params="id supporting_network supporting_node supporting_tp">
         <nt:termination-point>
@@ -43,3 +36,12 @@
         </nt:termination-point>
     </xacro:macro>
+    <xacro:macro name="wifi6_L1" params="id connector_type connector_format">
+        <nt:termination-point>
+            <nt:tp-id>${id}</nt:tp-id>
+            <l1t:l1-termination-point-attributes>
+                <l1t:connector-type>${connector_type}</l1t:connector-type>
+                <l1t:connector-format>${connector_format}</l1t:connector-format>
+            </l1t:l1-termination-point-attributes>
+        </nt:termination-point>
+    </xacro:macro>
 </robot>
