Commit message: nw iface descr added

File: network-components/interface_description/urdf/wifi4.urdf.xacro (robot description, xacro)
@@ -1,10 +1,11 @@
 <?xml version="1.0" encoding="UTF-8" ?>
 <robot xmlns:xacro="http://ros.org/wiki/xacro"
-       xmlns:robot-network-topology="urn:ietf:params:xml:ns:yang:robot-network-topology"
-       xmlns:layer1="urn:ietf:params:xml:ns:yang:layer1"
-       xmlns:layer2="urn:ietf:params:xml:ns:yang:layer2"
+       xmlns:ietf-network-topology="urn:ietf:params:xml:ns:yang:ietf-network-topology"
+       xmlns:device-layer="urn:ietf:params:xml:ns:yang:device-layer"
+       xmlns:network-layer="urn:ietf:params:xml:ns:yang:network-layer"
        name="wifi4">
-    <xacro:property name="wifi4_yaml_file" value="$(find interface-description)/config/wifi4.yaml" />
+    <xacro:property name="wifi4_yaml_file" value="$(find interface_description)/config/wifi4.yaml" />
     <xacro:property name="wifi4_props" value="${xacro.load_yaml(wifi4_yaml_file)}"/>
+    <xacro:property name="wifi4_type" value="${wifi4_props['wireless-connection']['type']}"/>
     <xacro:property name="wifi4_length" value="${wifi4_props['wireless-connection']['length']}"/>
     <xacro:property name="wifi4_bandwidth" value="${wifi4_props['wireless-connection']['bandwidth']}"/>
@@ -22,5 +23,5 @@
     <xacro:macro name="wifi4" params="parent L2_network_id L1_network_id L2_id:=wifi4_L2 L1_id:=wifi4_L1"/>
     <xacro:macro name="wifi4_L2" params="id supporting_network supporting_node supporting_tp">
-        <robot-network-topology:termination-point>
+        <ietf-network-topology:termination-point>
             <tp-id>${id}</tp-id>
             <supporting-termination-point>
@@ -29,18 +30,22 @@
                 <tp-ref>${supporting_tp}</tp-ref>
             </supporting-termination-point>
-            <layer2:l2-termination-point-attributes>
+            <network-layer:network-layer-termination-point-attributes>
+                <tp-type>${wifi4_type}</tp-type>
                 <bandwidth>${wifi4_bandwidth}</bandwidth>
                 <jitter>${wifi4_jitter}</jitter>
-            </layer2:l2-termination-point-attributes>
-        </robot-network-topology:termination-point>
+                <packet_loss>${wifi4_packet_loss}</packet_loss>
+                <reliability>${wifi4_reliability}</reliability>
+                <cost>${wifi4_cost}</cost>
+            </network-layer:network-layer-termination-point-attributes>
+        </ietf-network-topology:termination-point>
     </xacro:macro>
     <xacro:macro name="wifi4_L1" params="id connector_type connector_format">
-        <robot-network-topology:termination-point>
+        <ietf-network-topology:termination-point>
             <tp-id>${id}</tp-id>
-            <layer1:l1-termination-point-attributes>
+            <device-layer:device-layer-termination-point-attributes>
                 <connector-type>${connector_type}</connector-type>
                 <connector-format>${connector_format}</connector-format>
-            </layer1:l1-termination-point-attributes>
-        </robot-network-topology:termination-point>
+            </device-layer:device-layer-termination-point-attributes>
+        </ietf-network-topology:termination-point>
     </xacro:macro>
 </robot>

File: network-components/interface_description/urdf/wifi5.urdf.xacro (robot description, xacro)
@@ -1,10 +1,11 @@
 <?xml version="1.0" encoding="UTF-8" ?>
 <robot xmlns:xacro="http://ros.org/wiki/xacro"
-       xmlns:robot-network-topology="urn:ietf:params:xml:ns:yang:robot-network-topology"
-       xmlns:layer1="urn:ietf:params:xml:ns:yang:layer1"
-       xmlns:layer2="urn:ietf:params:xml:ns:yang:layer2"
+       xmlns:ietf-network-topology="urn:ietf:params:xml:ns:yang:ietf-network-topology"
+       xmlns:device-layer="urn:ietf:params:xml:ns:yang:device-layer"
+       xmlns:network-layer="urn:ietf:params:xml:ns:yang:network-layer"
        name="wifi5">
-    <xacro:property name="wifi5_yaml_file" value="$(find interface-description)/config/wifi5.yaml" />
+    <xacro:property name="wifi5_yaml_file" value="$(find interface_description)/config/wifi5.yaml" />
     <xacro:property name="wifi5_props" value="${xacro.load_yaml(wifi5_yaml_file)}"/>
+    <xacro:property name="wifi5_type" value="${wifi5_props['wireless-connection']['type']}"/>
     <xacro:property name="wifi5_length" value="${wifi5_props['wireless-connection']['length']}"/>
     <xacro:property name="wifi5_bandwidth" value="${wifi5_props['wireless-connection']['bandwidth']}"/>
@@ -22,5 +23,5 @@
     <xacro:macro name="wifi5" params="parent L2_network_id L1_network_id L2_id:=wifi5_L2 L1_id:=wifi5_L1"/>
     <xacro:macro name="wifi5_L2" params="id supporting_network supporting_node supporting_tp">
-        <robot-network-topology:termination-point>
+        <ietf-network-topology:termination-point>
             <tp-id>${id}</tp-id>
             <supporting-termination-point>
@@ -29,18 +30,22 @@
                 <tp-ref>${supporting_tp}</tp-ref>
             </supporting-termination-point>
-            <layer2:l2-termination-point-attributes>
+            <network-layer:network-layer-termination-point-attributes>
+                <tp-type>${wifi5_type}</tp-type>
                 <bandwidth>${wifi5_bandwidth}</bandwidth>
                 <jitter>${wifi5_jitter}</jitter>
-            </layer2:l2-termination-point-attributes>
-        </robot-network-topology:termination-point>
+                <packet_loss>${wifi5_packet_loss}</packet_loss>
+                <reliability>${wifi5_reliability}</reliability>
+                <cost>${wifi5_cost}</cost>
+            </network-layer:network-layer-termination-point-attributes>
+        </ietf-network-topology:termination-point>
     </xacro:macro>
     <xacro:macro name="wifi5_L1" params="id connector_type connector_format">
-        <robot-network-topology:termination-point>
+        <ietf-network-topology:termination-point>
             <tp-id>${id}</tp-id>
-            <layer1:l1-termination-point-attributes>
+            <device-layer:device-layer-termination-point-attributes>
                 <connector-type>${connector_type}</connector-type>
                 <connector-format>${connector_format}</connector-format>
-            </layer1:l1-termination-point-attributes>
-        </robot-network-topology:termination-point>
+            </device-layer:device-layer-termination-point-attributes>
+        </ietf-network-topology:termination-point>
     </xacro:macro>
 </robot>

File: network-components/interface_description/urdf/wifi6.urdf.xacro (robot description, xacro)
@@ -1,10 +1,11 @@
 <?xml version="1.0" encoding="UTF-8" ?>
 <robot xmlns:xacro="http://ros.org/wiki/xacro"
-       xmlns:robot-network-topology="urn:ietf:params:xml:ns:yang:robot-network-topology"
-       xmlns:layer1="urn:ietf:params:xml:ns:yang:layer1"
-       xmlns:layer2="urn:ietf:params:xml:ns:yang:layer2"
+       xmlns:ietf-network-topology="urn:ietf:params:xml:ns:yang:ietf-network-topology"
+       xmlns:device-layer="urn:ietf:params:xml:ns:yang:device-layer"
+       xmlns:network-layer="urn:ietf:params:xml:ns:yang:network-layer"
        name="wifi6">
-    <xacro:property name="wifi6_yaml_file" value="$(find interface-description)/config/wifi6.yaml" />
+    <xacro:property name="wifi6_yaml_file" value="$(find interface_description)/config/wifi6.yaml" />
     <xacro:property name="wifi6_props" value="${xacro.load_yaml(wifi6_yaml_file)}"/>
+    <xacro:property name="wifi6_type" value="${wifi6_props['wireless-connection']['type']}"/>
     <xacro:property name="wifi6_length" value="${wifi6_props['wireless-connection']['length']}"/>
     <xacro:property name="wifi6_bandwidth" value="${wifi6_props['wireless-connection']['bandwidth']}"/>
@@ -22,5 +23,5 @@
     <xacro:macro name="wifi6" params="parent L2_network_id L1_network_id L2_id:=wifi6_L2 L1_id:=wifi6_L1"/>
     <xacro:macro name="wifi6_L2" params="id supporting_network supporting_node supporting_tp">
-        <robot-network-topology:termination-point>
+        <ietf-network-topology:termination-point>
             <tp-id>${id}</tp-id>
             <supporting-termination-point>
@@ -29,18 +30,23 @@
                 <tp-ref>${supporting_tp}</tp-ref>
             </supporting-termination-point>
-            <layer2:l2-termination-point-attributes>
+            <network-layer:network-layer-termination-point-attributes>
+                <tp-type>${wifi6_type}</tp-type>
                 <bandwidth>${wifi6_bandwidth}</bandwidth>
                 <jitter>${wifi6_jitter}</jitter>
-            </layer2:l2-termination-point-attributes>
-        </robot-network-topology:termination-point>
+                <jitter>${wifi6_packet_loss}</jitter>
+                <packet_loss>${wifi6_packet_loss}</packet_loss>
+                <reliability>${wifi6_reliability}</reliability>
+                <cost>${wifi6_cost}</cost>
+            </network-layer:network-layer-termination-point-attributes>
+        </ietf-network-topology:termination-point>
     </xacro:macro>
     <xacro:macro name="wifi6_L1" params="id connector_type connector_format">
-        <robot-network-topology:termination-point>
+        <ietf-network-topology:termination-point>
             <tp-id>${id}</tp-id>
-            <layer1:l1-termination-point-attributes>
+            <device-layer:device-layer-termination-point-attributes>
                 <connector-type>${connector_type}</connector-type>
                 <connector-format>${connector_format}</connector-format>
-            </layer1:l1-termination-point-attributes>
-        </robot-network-topology:termination-point>
+            </device-layer:device-layer-termination-point-attributes>
+        </ietf-network-topology:termination-point>
     </xacro:macro>
 </robot>
