Commit message: namespaces updated, interfaces added

File: network-components/flightrack_description/urdf/flightrack.urdf.xacro (robot description, xacro)
@@ -1,11 +1,11 @@
 <?xml version="1.0" encoding="UTF-8" ?>
 <robot xmlns:xacro="http://ros.org/wiki/xacro"
-       xmlns:nw="urn:network"
-       xmlns:nt="urn:network-topology"
+       xmlns:nw="urn:robot-network"
+       xmlns:nt="urn:robot-network-topology"
        xmlns:l1t="urn:layer1"
        xmlns:l2t="urn:layer2"
        name="flightrack">
     <xacro:include filename="$(find interface-description)/urdf/cat6.urdf.xacro"/>
-    <xacro:macro name="flightrack" params="parent L2_network_id:=Data_Link L1_network_id:=Physical L2_id:=Flightrack_L2 L1_id:=Flightrack_L1">
+    <xacro:macro name="flightrack" params="parent L2_network_id:=network_level L1_network_id:=device_level L2_id:=flightrack_L2 L1_id:=flightrack_L1">
         <joint name="flightrack_joint" type="fixed">
             <origin xyz="-2 2 0" rpy="1.57 0 1.57" />
@@ -64,9 +64,9 @@
                         <l1t:device-type>switch</l1t:device-type>
                     </l1t:l1-node-attributes>
-                    <xacro:cat6_L1 id="eth_1"/>
-                    <xacro:cat6_L1 id="eth_2"/>
-                    <xacro:cat6_L1 id="eth_3"/>
-                    <xacro:cat6_L1 id="eth_4"/>
-                    <xacro:cat6_L1 id="eth_5"/>
+                    <xacro:cat6_L1 id="eth_1" connector_type="rj45" connector_format="female"/>
+                    <xacro:cat6_L1 id="eth_2" connector_type="rj45" connector_format="female"/>
+                    <xacro:cat6_L1 id="eth_3" connector_type="rj45" connector_format="female"/>
+                    <xacro:cat6_L1 id="eth_4" connector_type="rj45" connector_format="female"/>
+                    <xacro:cat6_L1 id="eth_5" connector_type="rj45" connector_format="female"/>
                 </nw:node>
             </nw:network>
