Commit message: yang in urdf updated

File: network-components/flightrack_description/urdf/flightrack.urdf.xacro (robot description, xacro)
@@ -1,14 +1,13 @@
 <?xml version="1.0" encoding="UTF-8" ?>
 <robot xmlns:xacro="http://ros.org/wiki/xacro"
-       xmlns:layer1="urn:ietf:params:xml:ns:yang:layer1"
        name="flightrack">
-    <xacro:include filename="$(find interface-description)/urdf/cat6.urdf.xacro"/>
-    <xacro:macro name="flightrack" params="parent L2_network_id:=network_level L1_network_id:=device_level L2_id:=flightrack_L2 L1_id:=flightrack_L1">
-        <joint name="flightrack_joint" type="fixed">
-            <origin xyz="-2 2 0" rpy="1.57 0 1.57" />
+    <xacro:include filename="$(find interface_description)/urdf/cat6.urdf.xacro"/>
+    <xacro:macro name="flightrack" params="parent id:=0  origin_xyz:='-2 2 0' origin_rpy:='1.57 0 1.57' ">
+        <joint name="flightrack_${id}_joint" type="fixed">
+            <origin xyz="${origin_xyz}" rpy="${origin_rpy}" />
             <parent link="${parent}"/>
-            <child link="flightrack_link"/>
+            <child link="flightrack_${id}_link"/>
         </joint>
-        <link name="flightrack_link">
+        <link name="flightrack_${id}_link">
             <visual>
                 <origin rpy="0 0 0" xyz="0 0 0"/>
@@ -27,41 +26,15 @@
             </collision>
         </link>
-        <yang>
-            <!-- Flightrack L2 network topology -->
-            <network>
-                <network-id>${L2_network_id}</network-id>
-                <supporting-network>
-                    <network-ref>${L1_network_id}</network-ref>
-                    <tf-parent>${parent}</tf-parent>
-                </supporting-network>
-                <node>
-                    <node-id>${L2_id}</node-id>
-                    <supporting-node>
-                        <network-ref>${L2_id}</network-ref>
-                        <node-ref>${L1_id}</node-ref>
-                    </supporting-node>
-                    <xacro:cat6_L2 id="eth_1" supporting_network="${L1_network_id}" supporting_node="${L1_id}" supporting_tp="eth_1"/>
-                    <xacro:cat6_L2 id="eth_2" supporting_network="${L1_network_id}" supporting_node="${L1_id}" supporting_tp="eth_2"/>
-                    <xacro:cat6_L2 id="eth_3" supporting_network="${L1_network_id}" supporting_node="${L1_id}" supporting_tp="eth_3"/>
-                    <xacro:cat6_L2 id="eth_4" supporting_network="${L1_network_id}" supporting_node="${L1_id}" supporting_tp="eth_4"/>
-                    <xacro:cat6_L2 id="eth_5" supporting_network="${L1_network_id}" supporting_node="${L1_id}" supporting_tp="eth_5"/>
-                </node>
-            </network>
-            <!-- Flightrack L1 network topology -->
-            <network>
-                <network-id>${L1_network_id}</network-id>
-                <node>
-                    <node-id>${L1_id}</node-id>
-                    <layer1:l1-node-attributes>
-                        <device-type>switch</device-type>
-                    </layer1:l1-node-attributes>
-                    <xacro:cat6_L1 id="eth_1" connector_type="rj45" connector_format="female"/>
-                    <xacro:cat6_L1 id="eth_2" connector_type="rj45" connector_format="female"/>
-                    <xacro:cat6_L1 id="eth_3" connector_type="rj45" connector_format="female"/>
-                    <xacro:cat6_L1 id="eth_4" connector_type="rj45" connector_format="female"/>
-                    <xacro:cat6_L1 id="eth_5" connector_type="rj45" connector_format="female"/>
-                </node>
-            </network>
-        </yang>
+        <!-- Flightrack network topology -->
+        <node>
+            <node-id>flightrack-${id}-node</node-id>
+            <dl:device-layer-node-attributes xmlns:dl="urn:ietf:params:xml:ns:yang:device-layer">
+                <dl:device-name>flightrack-${id}</dl:device-name>
+                <dl:device-type>flightrack</dl:device-type>
+                <dl:device-weight>15000</dl:device-weight>
+            </dl:device-layer-node-attributes>
+            <xacro:cat6 parent="flightrack_${id}_link" prefix="flightrack_${id}" id="0" origin_xyz="0.04 0.068 0.032" origin_rpy="-1.5707963 0 0" />
+            <xacro:cat6 parent="flightrack_${id}_link" prefix="flightrack_${id}" id="1" origin_xyz="0.05 0.068 0.032" origin_rpy="-1.5707963 0 0" />
+        </node>
     </xacro:macro>
 </robot>

File: network-components/nuc_description/urdf/nuc.urdf.xacro (robot description, xacro)
@@ -1,17 +1,14 @@
 <?xml version="1.0"?>
 <robot xmlns:xacro="http://ros.org/wiki/xacro"
-       xmlns:layer1="urn:ietf:params:xml:ns:yang:layer1"
        name="nuc">
-    <xacro:include filename="$(find interface-description)/urdf/cat6.urdf.xacro"/>
-    <xacro:include filename="$(find interface-description)/urdf/usb30.urdf.xacro"/>
-    <xacro:include filename="$(find interface-description)/urdf/wifi5.urdf.xacro"/>
-    <xacro:macro name="nuc" params="parent L2_network_id:=network_level L1_network_id:=device_level L2_id:=nuc_L2 L1_id:=nuc_L1">
-    <!-- <xacro:macro name="nuc" params="parent L1_id L2_id L1_network_id L2_network_id"> -->
-        <joint name="nuc_joint" type="fixed">
-            <origin xyz="-1 1 0" rpy="0 0 0" />
+    <xacro:include filename="$(find interface_description)/urdf/cat6.urdf.xacro"/>
+    <xacro:include filename="$(find interface_description)/urdf/usb30.urdf.xacro"/>
+    <xacro:macro name="nuc" params="parent id:=0 origin_xyz:='-1 1 0' origin_rpy:='0 0 0' ">
+        <joint name="nuc-${id}-joint" type="fixed">
+            <origin xyz="${origin_xyz}" rpy="${origin_rpy}" />
             <parent link="${parent}"/>
-            <child link="nuc_link"/>
+            <child link="nuc-${id}-link"/>
         </joint>
-        <link name="nuc_link">
+        <link name="nuc-${id}-link">
             <visual>
                 <origin rpy="0 0 0" xyz="0 0 0"/>
@@ -30,45 +27,16 @@
             </collision>
         </link>
-        <yang>
-            <!-- NUC L2 network topology -->
-            <network>
-                <network-id>${L2_network_id}</network-id>
-                <supporting-network>
-                    <network-ref>${L1_network_id}</network-ref>
-                    <tf-parent>${parent}</tf-parent>
-                </supporting-network>
-                <node>
-                    <node-id>${L2_id}</node-id>
-                    <supporting-node>
-                        <network-ref>${L2_id}</network-ref>
-                        <node-ref>${L1_id}</node-ref>
-                    </supporting-node>
-                    <xacro:usb30_L2 id="usb_1" supporting_network="${L1_network_id}" supporting_node="${L1_id}" supporting_tp="usb_1"/>
-                    <xacro:usb30_L2 id="usb_2" supporting_network="${L1_network_id}" supporting_node="${L1_id}" supporting_tp="usb_2"/>
-                    <xacro:usb30_L2 id="usb_3" supporting_network="${L1_network_id}" supporting_node="${L1_id}" supporting_tp="usb_3"/>
-                    <xacro:usb30_L2 id="usb_4" supporting_network="${L1_network_id}" supporting_node="${L1_id}" supporting_tp="usb_3"/>
-                    <xacro:usb30_L2 id="usb_5" supporting_network="${L1_network_id}" supporting_node="${L1_id}" supporting_tp="usb_3"/>
-                    <xacro:cat6_L2 id="eth_1" supporting_network="${L1_network_id}" supporting_node="${L1_id}" supporting_tp="eth_1"/>
-                    <xacro:wifi5_L2 id="wireless_1" supporting_network="${L1_network_id}" supporting_node="${L1_id}" supporting_tp="wireless_1"/>
-                </node>
-            </network>
-            <!-- NUC L1 network topology -->
-            <network>
-                <network-id>${L1_network_id}</network-id>
-                <node>
-                    <node-id>${L1_id}</node-id>
-                    <layer1:l1-node-attributes>
-                        <device-type>pc</device-type>
-                    </layer1:l1-node-attributes>
-                    <xacro:usb30_L1 id="usb_1" connector_type="usb-std_A" connector_format="female"/>
-                    <xacro:usb30_L1 id="usb_2" connector_type="usb-std_A" connector_format="female"/>
-                    <xacro:usb30_L1 id="usb_3" connector_type="usb-std_A" connector_format="female"/>
-                    <xacro:usb30_L1 id="usb_4" connector_type="usb-type_C" connector_format="female"/>
-                    <xacro:usb30_L1 id="usb_5" connector_type="usb-type_C" connector_format="female"/>
-                    <xacro:cat6_L1 id="eth_1" connector_type="rj45" connector_format="female"/>
-                    <!-- <xacro:wifi5_L1 id="wireless_1" connector-type="wireless" connector_format="wireless"/> -->
-                </node>
-            </network>
-        </yang>
+        <!-- NUC network topology -->
+        <node>
+            <node-id>nuc-${id}-node</node-id>
+            <dl:device-layer-node-attributes xmlns:dl="urn:ietf:params:xml:ns:yang:device-layer">
+                <dl:device-name>nuc-${id}</dl:device-name>
+                <dl:device-type>pc</dl:device-type>
+                <dl:weight>1000</dl:weight>
+            </dl:device-layer-node-attributes>
+            <xacro:cat6 parent="nuc-${id}-link" prefix="nuc-${id}" id="0" origin_xyz="0.04 0.068 0.032" origin_rpy="-1.5707963 0 0"/>
+            <xacro:usb30 parent="nuc-${id}-link" prefix="nuc-${id}" id="0" origin_xyz="0.087 0.119 0.019" origin_rpy="1.57 1.57 0"/>
+            <xacro:usb30 parent="nuc-${id}-link" prefix="nuc-${id}" id="1" origin_xyz="0.075 0.119 0.0199" origin_rpy="1.57 1.57 0"/>
+        </node>
     </xacro:macro>
 </robot>

File: network-components/nw-5g-modem_description/urdf/nw-5g-modem.urdf.xacro (robot description, xacro)
@@ -1,15 +1,14 @@
 <?xml version="1.0" encoding="UTF-8" ?>
 <robot xmlns:xacro="http://ros.org/wiki/xacro"
-       xmlns:layer1="urn:ietf:params:xml:ns:yang:layer1"
        name="nw-5g-modem">
-    <xacro:include filename="$(find interface-description)/urdf/usb30.urdf.xacro" />
-    <xacro:include filename="$(find interface-description)/urdf/nw_5g_rel15.urdf.xacro"/>
-    <xacro:macro name="nw-5g-modem" params=" parent L2_network_id:=network_level L1_network_id:=device_level L2_id:=nw_5g_modem_L2 L1_id:=nw_5g_modem_L1">
-        <joint name="nw-5g-modem_joint" type="fixed">
-            <origin xyz="-1 1.2 0" rpy="0 0 3.14" />
+    <xacro:include filename="$(find interface_description)/urdf/usb30.urdf.xacro" />
+    <!-- <xacro:include filename="$(find interface_description)/urdf/nw_5g_rel15.urdf.xacro"/> -->
+    <xacro:macro name="nw-5g-modem" params="parent id:=0 origin_xyz:='-1 1.2 0' origin_rpy:='0 0 3.14' ">
+        <joint name="nw-5g-modem_${id}_joint" type="fixed">
+            <origin xyz="${origin_xyz}" rpy="${origin_rpy}" />
             <parent link="${parent}"/>
-            <child link="nw-5g-modem_link"/>
+            <child link="nw-5g-modem-${id}-link"/>
         </joint>
-        <link name="nw-5g-modem_link">
+        <link name="nw-5g-modem-${id}-link">
             <visual>
                 <origin rpy="0 0 0" xyz="0 0 0"/>
@@ -28,35 +27,13 @@
             </collision>
         </link>
-        <yang>
-            <!-- 5gmodem L2 network topology -->
-            <network>
-                <network-id>${L2_network_id}</network-id>
-                <supporting-network>
-                    <network-ref>${L1_network_id}</network-ref>
-                    <tf-parent>${parent}</tf-parent>
-                </supporting-network>
-                <node>
-                    <node-id>${L2_id}</node-id>
-                    <supporting-node>
-                        <network-ref>${L1_network_id}</network-ref>
-                        <node-ref>${L1_id}</node-ref>
-                    </supporting-node>
-                    <xacro:usb30_L2 id="usb_1" supporting_network="${L1_network_id}" supporting_node="${L1_id}" supporting_tp="usb_1"/>
-                    <xacro:nw_5g_rel15_L2 id="wireless_1" supporting_network="${L1_network_id}" supporting_node="${L1_id}" supporting_tp="wireless_1"/>
-                </node>
-            </network>
-            <!-- 5gmodem L1 network topology -->
-            <network>
-                <network-id>${L1_network_id}</network-id>
-                <node>
-                    <node-id>${L1_id}</node-id>
-                    <layer1:l1-node-attributes>
-                        <device-type>nw-5g-modem</device-type>
-                    </layer1:l1-node-attributes>
-                    <xacro:usb30_L1 id="usb_1" connector_type="usb-std_A" connector_format="female"/>
-                    <xacro:nw_5g_rel15_L1 id="wireless_1" connector_type="wireless" connector_format="wireless"/>
-                </node>
-            </network>
-        </yang>
+        <node>
+            <node-id>nw-5g-modem-${id}-node</node-id>
+            <dl:device-layer-node-attributes xmlns:dl="urn:ietf:params:xml:ns:yang:device-layer">
+                <dl:device-name>nw-5g-modem-${id}</dl:device-name>
+                <dl:device-type>modem</dl:device-type>
+            </dl:device-layer-node-attributes>
+            <xacro:cat6 parent="nw-5g-modem-${id}-link" prefix="nw-5g-modem-${id}" id="0" origin_xyz="0.0 0.1 0.2" origin_rpy="-1.57 0 0"/>
+            <xacro:usb30 parent="nw-5g-modem-${id}-link" prefix="nw-5g-modem-${id}" id="0" origin_xyz="0 0.044 0" origin_rpy="1.57 0 0"/>
+        </node>
     </xacro:macro>
 </robot>

File: network-components/poesw_description/urdf/poe-switch.urdf.xacro (robot description, xacro)
@@ -1,14 +1,13 @@
 <?xml version="1.0" encoding="UTF-8" ?>
 <robot xmlns:xacro="http://ros.org/wiki/xacro"
-       xmlns:layer1="urn:ietf:params:xml:ns:yang:layer1"
        name="poesw">
-    <xacro:include filename="$(find interface-description)/urdf/cat6.urdf.xacro"/>
-    <xacro:macro name="poesw" params="parent L2_network_id:=network_level L1_network_id:=device_level L2_id:=poesw_L2 L1_id:=poesw_L1">
-        <joint name="poeswitch_joint" type="fixed">
-            <origin xyz="-1 1.5 0" rpy="0 0 0" />
+    <xacro:include filename="$(find interface_description)/urdf/cat6.urdf.xacro"/>
+    <xacro:macro name="poesw" params="parent id:=0 origin_xyz:='-1 1.5 0' origin_rpy:='0 0 0' ">
+        <joint name="poesw-${id}-joint" type="fixed">
+            <origin xyz="${origin_xyz}" rpy="${origin_rpy}"/>
             <parent link="${parent}"/>
-            <child link="poeswitch_link"/>
+            <child link="poesw-${id}-link"/>
         </joint>
-        <link name="poeswitch_link">
+        <link name="poesw-${id}-link">
             <visual>
                 <origin rpy="0 0 0" xyz="0 0 0"/>
@@ -27,41 +26,18 @@
             </collision>
         </link>
-        <yang>
-            <!-- POE Switch L2 network topology -->
-            <network>
-                <network-id>${L2_network_id}</network-id>
-                <supporting-network>
-                    <network-ref>${L1_network_id}</network-ref>
-                    <tf-parent>${parent}</tf-parent>
-                </supporting-network>
-                <node>
-                    <node-id>${L2_id}</node-id>
-                    <supporting-node>
-                        <network-ref>${L2_id}</network-ref>
-                        <node-ref>${L1_id}</node-ref>
-                    </supporting-node>
-                    <xacro:cat6_L2 id="eth_1" supporting_network="${L1_network_id}" supporting_node="${L1_id}" supporting_tp="eth_1"/>
-                    <xacro:cat6_L2 id="eth_2" supporting_network="${L1_network_id}" supporting_node="${L1_id}" supporting_tp="eth_2"/>
-                    <xacro:cat6_L2 id="eth_3" supporting_network="${L1_network_id}" supporting_node="${L1_id}" supporting_tp="eth_3"/>
-                    <xacro:cat6_L2 id="eth_4" supporting_network="${L1_network_id}" supporting_node="${L1_id}" supporting_tp="eth_4"/>
-                    <xacro:cat6_L2 id="eth_5" supporting_network="${L1_network_id}" supporting_node="${L1_id}" supporting_tp="eth_5"/>
-                </node>
-            </network>
-            <!-- POE Switch L1 network topology -->
-            <network>
-                <network-id>${L1_network_id}</network-id>
-                <node>
-                    <node-id>${L1_id}</node-id>
-                    <layer1:l1-node-attributes>
-                        <device-type>switch</device-type>
-                    </layer1:l1-node-attributes>
-                    <xacro:cat6_L1 id="eth_1" connector_type="rj45" connector_format="female"/>
-                    <xacro:cat6_L1 id="eth_2" connector_type="rj45" connector_format="female"/>
-                    <xacro:cat6_L1 id="eth_3" connector_type="rj45" connector_format="female"/>
-                    <xacro:cat6_L1 id="eth_4" connector_type="rj45" connector_format="female"/>
-                    <xacro:cat6_L1 id="eth_5" connector_type="rj45" connector_format="female"/>
-                </node>
-            </network>
-        </yang>
+        <!-- poe-switch network topology -->
+        <node>
+            <node-id>poesw-${id}-node</node-id>
+            <dl:device-layer-node-attributes xmlns:dl="urn:ietf:params:xml:ns:yang:device-layer">
+                <dl:device-name>poesw-${id}</dl:device-name>
+                <dl:device-type>switch</dl:device-type>
+                <dl:device-weight>230</dl:device-weight>
+            </dl:device-layer-node-attributes>
+            <xacro:cat6 parent="poesw-${id}-link" prefix="poesw-${id}" id="0" origin_xyz="-0.014 0.002 0" origin_rpy="1.5707963 0 0"/>
+            <xacro:cat6 parent="poesw-${id}-link" prefix="poesw-${id}" id="1" origin_xyz="0.002 0.002 0" origin_rpy="1.5707963 0 0"/>
+            <xacro:cat6 parent="poesw-${id}-link" prefix="poesw-${id}" id="2" origin_xyz="0.018 0.002 0" origin_rpy="1.5707963 0 0"/>
+            <xacro:cat6 parent="poesw-${id}-link" prefix="poesw-${id}" id="3" origin_xyz="0.034 0.002 0" origin_rpy="1.5707963 0 0"/>
+            <xacro:cat6 parent="poesw-${id}-link" prefix="poesw-${id}" id="4" origin_xyz="0.05 0.002 0" origin_rpy="1.5707963 0 0"/>
+        </node>
     </xacro:macro>
 </robot>

File: network-components/radiodot_description/urdf/radiodot.urdf.xacro (robot description, xacro)
@@ -1,15 +1,14 @@
 <?xml version="1.0" encoding="UTF-8" ?>
 <robot xmlns:xacro="http://ros.org/wiki/xacro"
-       xmlns:layer1="urn:ietf:params:xml:ns:yang:layer1"
        name="radiodot">
-    <xacro:include filename="$(find interface-description)/urdf/cat6.urdf.xacro"/>
-    <xacro:include filename="$(find interface-description)/urdf/nw_5g_rel15.urdf.xacro"/>
-    <xacro:macro name="radiodot" params="parent L2_network_id:=network_level L1_network_id:=device_level L2_id:=radiobot_L2 L1_id:=radiobot_L1">
-        <joint name="radiodot_joint" type="fixed">
-            <origin xyz="-1 1.2 2" rpy="0 0 0" />
+    <xacro:include filename="$(find interface_description)/urdf/cat6.urdf.xacro"/>
+    <!-- <xacro:include filename="$(find interface_description)/urdf/nw_5g_rel15.urdf.xacro"/> -->
+    <xacro:macro name="radiodot" params="parent id:=0 origin_xyz:='0 2 0' origin_rpy:='0 0 0' ">
+        <joint name="radiodot-${id}-joint" type="fixed">
+            <origin xyz="${origin_xyz}" rpy="${origin_rpy}" />
             <parent link="${parent}"/>
-            <child link="radiodot_link"/>
+            <child link="radiodot-${id}-link"/>
         </joint>
-        <link name="radiodot_link">
+        <link name="radiodot-${id}-link">
             <visual>
                 <origin rpy="0 0 0" xyz="0 0 0"/>
@@ -28,33 +27,14 @@
             </collision>
         </link>
-        <yang>
-            <!-- radiodot L2 network topology -->
-            <network>
-                <network-id>${L2_network_id}</network-id>
-                <supporting-network>
-                    <network-ref>${L1_network_id}</network-ref>
-                    <tf-parent>${parent}</tf-parent>
-                </supporting-network>
-                <node>
-                    <node-id>${L2_id}</node-id>
-                    <supporting-node>
-                        <network-ref>${L2_id}</network-ref>
-                        <node-ref>${L1_id}</node-ref>
-                    </supporting-node>
-                    <xacro:cat6_L2 id="eth_1" supporting_network="${L1_network_id}" supporting_node="${L1_id}" supporting_tp="eth_1"/>
-                </node>
-            </network>
-            <!-- radiodot L1 network topology -->
-            <network>
-                <network-id>${L1_network_id}</network-id>
-                <node>
-                    <node-id>${L1_id}</node-id>
-                    <layer1:l1-node-attributes>
-                        <device-type>radiodot</device-type>
-                    </layer1:l1-node-attributes>
-                    <xacro:cat6_L1 id="eth_1" connector_type="rj45" connector_format="female"/>
-                </node>
-            </network>
-        </yang>
+        <!-- radiodot network topology -->
+        <node>
+            <node-id>radiodot-${id}-node</node-id>
+            <dl:device-layer-node-attributes xmlns:dl="urn:ietf:params:xml:ns:yang:device-layer">
+                <dl:device-name>radiodot-${id}</dl:device-name>
+                <dl:device-type>radiodot</dl:device-type>
+                <dl:device-weight>500</dl:device-weight>
+            </dl:device-layer-node-attributes>
+            <xacro:cat6 parent="radiodot-${id}-link" prefix="radiodot-${id}" id="0" origin_xyz="0 0 0" origin_rpy="0 0 0"/>
+        </node>
     </xacro:macro>
 </robot>
